File: minirov.brd (EAGLE design)
At the start: 65.8 x 51.6 mm, 66 parts, among them Q1 DMN6140L-13DICT-ND, Q2 DMN6140L-13DICT-ND, U1 DRV8848PWP, U2 DRV8848PWP, U4 S811-1X1T-06-F, Y1 ABM8-25.000MHZ-B2-T

Commit message: Cleaned up routing, moved some connectors
Parts:
- moved J8 30.5 mm to (62.2, 31.0)
- moved C2 20.9 mm to (14.8, 5.87)
- moved C3 20.9 mm to (14.8, 10.6)
- moved C15 20.9 mm to (23.5, 33.3)
- moved J12 20.9 mm to (2.24, 36.6)
- moved J21 20.9 mm to (4.78, 36.6)
- moved Q1 20.9 mm to (12.3, 32.8)
- moved C1 20.9 mm to (19.5, 41.1)
- moved C8 20.9 mm to (5.03, 6.68), turned to 139 degrees
- moved J11 20.9 mm to (2.11, 41.7)
- moved J15 20.9 mm to (4.65, 39.2)
- moved J18 20.9 mm to (12.0, 23.0)
- moved J19 20.9 mm to (14.8, 23.0)
- moved J3 20.9 mm to (24.7, 22.5)
- moved J4 20.9 mm to (27.4, 22.5)
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Routing:
- net N$4: track 0.00 -> 2.05 mm
- net +3V3: track 200.7 -> 202.7 mm
- net N$5: track 0.00 -> 1.91 mm
- net N$9: track 0.00 -> 1.81 mm
- net N$3: track 0.00 -> 1.59 mm
- net +5V: track 94.5 -> 95.8 mm
- net GND: vias 4 -> 25
